File: hardware/uMIDI.kicad_pcb (KiCad board)
At the start: 2 copper layers, 24.7 x 108 mm, 40 parts, among them IC1 ATTINY84, IC2 MCP4822, J1 USB, J2 CONN_01X02_MALE, J3 CONN_01X02_MALE, J4 CONN_01X02_MALE, Q1 20 MHz, T1 TESTPIN, T2 TESTPIN, T3 TESTPIN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

Commit message: license info added
Other:
- board text added: "CC-BY-SA"
- board text added: "uMIDI MK1 - seismic industries"
Changed lines of the file:
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@@
     (area -14.800001 -0.100001 10.100001 108.100001)
     (thickness 1.6)
-    (drawings 123)
+    (drawings 125)
     (tracks 560)
     (zones 0)
@@
       (net 23 "Net-(R6-Pad2)"))
   )
+  (gr_text "uMIDI MK1 - seismic industries" (at 1.5 32 90) (layer B.SilkS)
+    (effects (font (size 1.5 1.5) (thickness 0.3)) (justify mirror))
+  )
+  (gr_text CC-BY-SA (at 5 80.5 90) (layer B.SilkS)
+    (effects (font (size 3 3) (thickness 0.6)) (justify mirror))
+  )
   (gr_line (start -9.7 7.85) (end -10.55 8.7) (layer B.Mask) (width 1))
